File: Schematics/STM32_MegaBlaster/STM32_MegaBlaster.sch (KiCad schematic (older format))
At the start: 19 parts, among them J1 SD_Card, J2 USB_B, U1 BluePill_STM32F103C, U10 LD1117S33TR_SOT223, U11 LM2596T-5, U12 I2C_OLED, U2 SN769486, U3 YM2612, U4 CH340G, U5 LTC6904, U6 LTC6904, U7 23LC1024, U8 TL062, U9 TPA3122D2

Commit message: Saving schematic. Nearly Complete
Parts:
- added C10, C11: 22pF, symbol device:C_Small
- added C12, C26, C6, C7, C9: 100nF, symbol device:C_Small
- added C13: 680uF, symbol device:CP1_Small
- added C14: 220uF, symbol device:CP1_Small
- added C15, C16: 1uF, symbol device:C_Small
- added C17: 68uF, symbol device:CP1_Small
- added C18: 100uF, symbol device:CP1_Small
- added C19: 220pF, symbol device:C_Small
- added C20, C21, C8: 10uF, symbol device:CP1_Small
- added C22, C23, C24, C25: 5.6nF, symbol device:C_Small
- added C27, C28, C29, C30: 1uF, symbol device:CP1_Small
- added C31, C32: 0.22uF, symbol device:C_Small
- added C33, C?: 68nF, symbol device:C_Small
- added C34, C?: 1000uF, symbol device:CP1_Small
- added D1: SS34, symbol device:D_Schottky_Small_ALT
- added J3: Barrel_Jack, symbol conn:Barrel_Jack
- added J?: JACK_TRS_6PINS, symbol 3_5_TRS_Jack:JACK_TRS_6PINS
- added L1, L2, L3: 33uH, symbol device:L_Small
- added L4, L5: 22uH, symbol device:L_Small
- added R1, R11, R24, R25, R26: 10k, symbol device:R
- added R10, R9: 51k, symbol device:R
- added R2, R3: 4.7k, symbol device:R
- added R27, R30, R6, R7, R8: 2.2k, symbol device:R
- added R28, R29: 33k, symbol device:R
- added R4, R5: 47k, symbol device:R
- added SW1: PREV, symbol switches:SW_Push_Dual
- added SW2: RAND, symbol switches:SW_Push_Dual
- added SW3: NEXT, symbol switches:SW_Push_Dual
- added SW4: OPTION, symbol switches:SW_Push_Dual
- added SW5: PWR_SWITCH, symbol switches:SW_SPST
- added SW6, SW7: MUTE_SN, symbol switches:SW_Push_SPDT
- added Y1: 12MHz, symbol device:Crystal_Small
- C5: renamed from C?; value C_Small -> 10nF
- U10: value LD1117S33TR_SOT223 -> LD1117S33
Connections:
- net +5V: now also U10.3 (VI), U11.4 (FB), C14.1, C15.2, C16.2, C7.1, L1.1, L3.1, R2.1, R3.1
- net AGND: now also U8.4 (V-), C17.2, C18.2, C26.1, L2.2, R5.2
- net AVCC: now also U8.8 (V+), C17.1, C26.2, L3.2, R4.1
- net GND: now also J2.4 (GND), U10.1 (GND), U11.3 (GND), U11.5 (~ON~/OFF), U12.1 (GND), U4.1 (GND), U7.4 (GND), U9.14 (GAIN1), U9.15 (GAIN0), U9.20 (PGNDL), U9.7 (AGND1), U9.8 (AGND2), C10.2, C11.2, C12.2, C13.2, C14.2, C15.1, C16.1, C19.2, C29.2, C30.2, C33.1, C6.1, C7.2, C8.2, C9.2, C?.1, D1.2 (A), J3.2, J3.3, L2.1, L5.2, R6.2, R7.2, R8.2, SW1.3, SW2.3, SW3.3, SW4.3, SW6.3 (C), SW7.1 (A)
- net I2C_SCL: now also U12.3 (SCL), R2.2
- net I2C_SDA: now also U12.4 (SDA), R3.2
- net MOL: now also C21.1, R8.1
- net MOR: now also C20.1, R7.1
- net RAM_CS: now also U7.1 (CS)
- net SN_OUT: now also SW6.1 (A)
- net NEXT: now reaches U1.14 (PB1)
- net NEXT: now also SW3.1
- net RAND: now reaches U1.15 (PB10_SCL2)
- net RAND: now also SW2.1
- net PREV: now reaches U1.16 (PB11_SDA2)
- net PREV: now also SW1.1
- net RAM_SCK: now reaches U1.22 (PB13_SCK2)
- net RAM_SCK: now also U7.6 (SCK)
- net RAM_MISO: now reaches U1.23 (PB14_MISO2)
- net RAM_MISO: now also U7.2 (SO/SIO1)
- net RAM_MOSI: now reaches U1.24 (PB15_MOSI2)
- net RAM_MOSI: now also U7.5 (SI/SIO0)
- net TX: now reaches U1.26 (PA9_TX1)
- net TX: now also U4.3 (RX)
- net RX: now reaches U1.27 (PA10_RX1)
- net RX: now also U4.2 (TX)
- net OPTION: now reaches U1.8 (PA3_RX2)
- net OPTION: now also SW4.1
- net at U4.16 (VCC): now also J2.1 (VBUS), C9.1
- net at U4.4 (V3): now also C12.1
- net at U4.5 (D+): now also J2.3 (D+)
- net at U4.6 (D): now also J2.2 (D-)
- net at U4.7 (XI): now also C10.1, Y1.1
- net at U4.8 (XO): now also C11.1, Y1.2
- net at U7.7 (HOLD): now also R1.2
- net +3V3: now reaches U7.8 (VCC)
- net +3V3: now also U10.2 (VO), U12.2 (VCC), C6.2, C8.1, R1.1
- net PRE_R: now reaches U8.1
- net PRE_R: now also C28.1, R28.1
- net at U8.2 (-): now also R24.1, R28.2
- net AVCC_DIV2: now reaches U8.3 (+)
- net AVCC_DIV2: now also U8.5 (+), C18.1, C22.1, C24.1, R4.2, R5.1
- net at U8.6 (-): now also R26.1, R29.2
- net PRE_L: now reaches U8.7
- net PRE_L: now also C27.1, R29.1
- net +12V: now reaches U9.1 (PVCCL)
- net +12V: now also U11.1 (VIN), U9.10 (PVCCR), U9.16 (AVCC2), U9.17 (AVCC1), U9.2 (/SD), C13.1, SW5.1 (A), SW7.3 (C)
- net at U9.11 (PGRNR): now also C?.1, C?.2
- net at U9.12 (ROUT): now also C32.1, L5.1
- net at U9.13 (BSR): now also C32.2
- net at U9.18 (BSL): now also C31.2
- net at U9.19 (LOUT): now also C31.1, L4.1
- net at U9.3 (MUTE): now also SW7.2 (B)
- net at U9.4 (LIN): now also C27.2
- net at U9.5 (RIN): now also C28.2
- net at U9.6 (BYPASS): now also C29.1
- net at U9.9 (VCLAMP): now also C30.1
- net at U11.2 (OUT): now also D1.1 (K), L1.2
- new net: J3.1, SW5.2 (B)
- new net: C19.1, R10.2, R6.1, R9.2, SW6.2 (B)
- new net: C20.2, R30.2
- new net: C21.2, R27.2
- new net: C22.2, C23.2, R10.1, R11.2, R30.1
- new net: C24.2, C25.2, R25.2, R27.1, R9.1
- new net: C23.1, R11.1, R24.2
- new net: C25.1, R25.1, R26.2
- new net: C33.2, C34.1, L4.2
- new net L_OUT: C34.2
- new net R_OUT: C?.2
- no-connect marks 6 -> 22
Other:
- note added: "4"
- moved on the sheet: C1, C2, C3, C4, C5, J1, J2, U1, U10, U11, U12, U2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

Commit message: Schematic complete. Now working on PCB
Parts:
- removed J?: JACK_TRS_6PINS, symbol 3_5_TRS_Jack:JACK_TRS_6PINS
- added J4: AMP_OUT, Connectors:PJ320E_3.5mm_Jack, symbol 3_5_TRS_Jack:JACK_TRS_6PINS
- added J5: LINE_LEVEL_OUT, Connectors:PJ320E_3.5mm_Jack, symbol 3_5_TRS_Jack:JACK_TRS_6PINS
- added R12, R14: 9.1k, Resistors_THT:R_Axial_DIN0207_L6.3mm_D2.5mm_P7.62mm_Horizontal, symbol device:R
- added R13, R15: 1.2k, Resistors_THT:R_Axial_DIN0207_L6.3mm_D2.5mm_P7.62mm_Horizontal, symbol device:R
- C1, C10, C11, C12, C19, C2, C26, C31, C32, C33, C4, C5, C6, C7, C9: footprint (none) -> Capacitors_THT:C_Disc_D3.0mm_W1.6mm_P2.50mm
- C13: footprint (none) -> Capacitors_THT:CP_Radial_D10.0mm_P5.00mm
- C14, C17: footprint (none) -> Capacitors_THT:CP_Radial_D6.3mm_P2.50mm
- C15, C16, C20, C21, C22, C23, C24, C25: footprint (none) -> Capacitors_THT:C_Disc_D4.7mm_W2.5mm_P5.00mm
- C18: footprint (none) -> Capacitors_THT:CP_Radial_D5.0mm_P2.00mm
- C27, C28, C29, C30, C8: footprint (none) -> Capacitors_THT:CP_Radial_D4.0mm_P1.50mm
- C3: footprint (none) -> Capacitors_THT:C_Axial_L22.0mm_D10.5mm_P27.50mm_Horizontal
- C34: footprint (none) -> Capacitors_THT:CP_Radial_D8.0mm_P2.50mm
- C35: renamed from C?; footprint (none) -> Capacitors_THT:C_Disc_D3.0mm_W1.6mm_P2.50mm
- C36: renamed from C?; footprint (none) -> Capacitors_THT:CP_Radial_D8.0mm_P2.50mm
- D1: footprint (none) -> Diodes:DO-214AB
- J3: footprint (none) -> Connectors:BARREL_JACK
- L1, L2, L3: footprint (none) -> Inductors_THT:L_Radial_D7.0mm_P3.00mm
- L4, L5: footprint (none) -> Inductors_THT:L_Radial_D8.7mm_P5.00mm_Fastron_07HCP
- R1, R10, R11, R2, R24, R25, R26, R27, R28, R29, R3, R30, R4, R5, R6, R7, R8, R9: footprint (none) -> Resistors_THT:R_Axial_DIN0207_L6.3mm_D2.5mm_P7.62mm_Horizontal
- SW1, SW2, SW3, SW4: footprint (none) -> Buttons_Switches_THT:SW_TH_Tactile_Omron_B3F-10xx
- SW5, SW6: footprint (none) -> Switches:1825115-1
- SW7: value MUTE_SN -> GLOBAL_MUTE; footprint (none) -> Switches:1825115-1
- Y1: footprint (none) -> Crystals:Crystal_HC49-U_Vertical
Connections:
- net I2C_SDA is gone; now on net I2C_SCL: R3.2, U1.35 (PB7_SDA1), U12.4 (SDA), U5.2 (SDI), U6.2 (SDI)
- net +3V3: now also J1.4 (VDD)
- net GND: now also J1.3 (VSS), J1.6 (VSS), J4.1 (S), J5.4 (SN), R13.1, R15.1
- net L_OUT: now also J4.2 (T), R14.1, R15.2
- net R_OUT: now also J4.3 (R), R12.1, R13.2
- net SD_SCK: now reaches U1.10 (PA5_SCK1)
- net SD_SCK: now also J1.5 (CLK)
- net SD_MISO: now reaches U1.11 (PA6_MISO1)
- net SD_MISO: now also J1.7 (DAT0)
- net SD_MOSI: now reaches U1.12 (PA7_MOSI1)
- net SD_MOSI: now also J1.2 (CMD)
- net SD_CS: now reaches U1.9 (PA4)
- net SD_CS: now also J1.1 (CD/DAT3)
- new net: J5.2 (T), R14.2
- new net: J5.3 (R), R12.2
Other:
- note added: "Amplification and output"
- note added: "Main Soundchips, CPU, RAM & COM"
- note added: "Power input and regulation"
- note added: "Pre-amp"
- note added: "User Input/Output"
- moved on the sheet: C1, C10, C11, C12, C13, C14, C15, C16, C17, C18, C19, C2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

Commit message: PCB near complete
Parts:
- removed J5: LINE_LEVEL_OUT, Connectors:PJ320E_3.5mm_Jack, symbol 3_5_TRS_Jack:JACK_TRS_6PINS
- removed R12, R14: 9.1k, Resistors_THT:R_Axial_DIN0207_L6.3mm_D2.5mm_P7.62mm_Horizontal, symbol device:R
- removed R13, R15: 1.2k, Resistors_THT:R_Axial_DIN0207_L6.3mm_D2.5mm_P7.62mm_Horizontal, symbol device:R
- removed SW7: GLOBAL_MUTE, Switches:1825115-1, symbol switches:SW_Push_SPDT
- added C37: 1000uF, Capacitors_THT:CP_Radial_D8.0mm_P2.50mm, symbol device:CP1_Small
- added RV1: POT_Dual, Potentiometers:Potentiometer_Alps_RK163_Double_Vertical, symbol device:POT_Dual
Connections:
- wire segments 224 -> 217
Other:
- moved on the sheet: J4
Changed lines of the file:
@@
 L power:+5V #PWR0103
 U 1 1 5ADDA485
-P 5550 2900
-F 0 "#PWR0103" H 5550 2750 50  0001 C CNN
-F 1 "+5V" H 5565 3073 50  0000 C CNN
-F 2 "" H 5550 2900 50  0001 C CNN
-F 3 "" H 5550 2900 50  0001 C CNN
-	1    5550 2900
+P 5550 2550
+F 0 "#PWR0103" H 5550 2400 50  0001 C CNN
+F 1 "+5V" H 5565 2723 50  0000 C CNN
+F 2 "" H 5550 2550 50  0001 C CNN
+F 3 "" H 5550 2550 50  0001 C CNN
+	1    5550 2550
 	1    0    0    -1
 $EndComp
@@
 U 1 1 5ADDB1F9
 P 5700 3150
-F 0 "C2" V 5471 3150 50  0000 C CNN
-F 1 "100nF" V 5562 3150 50  0000 C CNN
+F 0 "C2" V 5500 3150 50  0000 C CNN
+F 1 "100nF" V 5600 3150 50  0000 C CNN
 F 2 "Capacitors_THT:C_Disc_D3.0mm_W1.6mm_P2.50mm" H 5700 3150 50  0001 C CNN
 F 3 "" H 5700 3150 50  0001 C CNN
@@
 Text GLabel 5200 3050 2    50   Input ~ 0
 YM_CLK
-Wire Wire Line
-	5550 2900 5550 3150
 Wire Wire Line
 	5550 3150 5600 3150
@@
 	0    1    1    0
 $EndComp
-$Comp
-L switches:SW_Push_SPDT SW7
-U 1 1 5AFD9689
-P 9800 2250
-F 0 "SW7" H 9800 2000 50  0000 C CNN
-F 1 "GLOBAL_MUTE" H 9750 2100 50  0000 C CNN
-F 2 "Switches:1825115-1" H 9800 2250 50  0001 C CNN
-F 3 "" H 9800 2250 50  0001 C CNN
-	1    9800 2250
-	-1   0    0    1
-$EndComp
 Wire Wire Line
 	10000 2250 10150 2250
@@
 Wire Wire Line
 	10150 2350 10300 2350
-$Comp
-L power:+12V #PWR02
-U 1 1 5AFF8DC1
-P 9550 2150
-F 0 "#PWR02" H 9550 2000 50  0001 C CNN
-F 1 "+12V" H 9565 2323 50  0000 C CNN
-F 2 "" H 9550 2150 50  0001 C CNN
-F 3 "" H 9550 2150 50  0001 C CNN
-	1    9550 2150
-	1    0    0    -1
-$EndComp
-Wire Wire Line
-	9550 2150 9600 2150
-$Comp
-L power:GND #PWR03
-U 1 1 5AFFF241
-P 9550 2350
-F 0 "#PWR03" H 9550 2100 50  0001 C CNN
-F 1 "GND" H 9555 2177 50  0000 C CNN
-F 2 "" H 9550 2350 50  0001 C CNN
-F 3 "" H 9550 2350 50  0001 C CNN
-	1    9550 2350
-	1    0    0    -1
-$EndComp
-Wire Wire Line
-	9550 2350 9600 2350
 Text GLabel 9950 2450 0    50   Input ~ 0
 PRE_L
@@
 L 3_5_TRS_Jack:JACK_TRS_6PINS J4
 U 1 1 5ADF760F
-P 15250 2450
-F 0 "J4" H 15231 2975 50  0000 C CNN
-F 1 "AMP_OUT" H 15231 2884 50  0000 C CNN
-F 2 "Connectors:PJ320E_3.5mm_Jack" H 15350 2300 50  0001 C CNN
-F 3 "" H 15350 2300 50  0001 C CNN
-	1    15250 2450
-	-1   0    0    1
-$EndComp
-$Comp
-L 3_5_TRS_Jack:JACK_TRS_6PINS J5
-U 1 1 5ADF76CD
 P 15250 4350
-F 0 "J5" H 15231 4875 50  0000 C CNN
-F 1 "LINE_LEVEL_OUT" H 15231 4784 50  0000 C CNN
+F 0 "J4" H 15231 4875 50  0000 C CNN
+F 1 "AMP_OUT" H 15231 4784 50  0000 C CNN
 F 2 "Connectors:PJ320E_3.5mm_Jack" H 15350 4200 50  0001 C CNN
 F 3 "" H 15350 4200 50  0001 C CNN
@@
 	-1   0    0    1
 $EndComp
-Text GLabel 14850 2250 0    50   Input ~ 0
+Text GLabel 13550 4000 0    50   Input ~ 0
 R_OUT
-Text GLabel 14850 2450 0    50   Input ~ 0
+Text GLabel 13550 4500 0    50   Input ~ 0
 L_OUT
 $Comp
 L power:GND #PWR011
 U 1 1 5ADF8747
-P 14750 2750
-F 0 "#PWR011" H 14750 2500 50  0001 C CNN
-F 1 "GND" H 14755 2577 50  0000 C CNN
-F 2 "" H 14750 2750 50  0001 C CNN
-F 3 "" H 14750 2750 50  0001 C CNN
-	1    14750 2750
-	1    0    0    -1
-$EndComp
-Wire Wire Line
-	14750 2750 14750 2650
-Wire Wire Line
-	14750 2650 14850 2650
-Wire Wire Line
-	14850 4650 14750 4650
-Wire Wire Line
-	14750 4650 14750 4750
-$Comp
-L power:GND #PWR014
-U 1 1 5AE0CA17
 P 14750 4750
-F 0 "#PWR014" H 14750 4500 50  0001 C CNN
+F 0 "#PWR011" H 14750 4500 50  0001 C CNN
 F 1 "GND" H 14755 4577 50  0000 C CNN
 F 2 "" H 14750 4750 50  0001 C CNN
@@
 	1    0    0    -1
 $EndComp
-$Comp
-L device:R R15
-U 1 1 5AE1B154
-P 13900 4850
-F 0 "R15" H 13970 4896 50  0000 L CNN
-F 1 "1.2k" V 13900 4750 50  0000 L CNN
-F 2 "Resistors_THT:R_Axial_DIN0207_L6.3mm_D2.5mm_P7.62mm_Horizontal" V 13830 4850 50  0001 C CNN
-F 3 "" H 13900 4850 50  0001 C CNN
-	1    13900 4850
-	-1   0    0    1
-$EndComp
-$Comp
-L device:R R13
-U 1 1 5AE1C030
-P 13600 4850
-F 0 "R13" H 13670 4896 50  0000 L CNN
-F 1 "1.2k" V 13600 4750 50  0000 L CNN
-F 2 "Resistors_THT:R_Axial_DIN0207_L6.3mm_D2.5mm_P7.62mm_Horizontal" V 13530 4850 50  0001 C CNN
-F 3 "" H 13600 4850 50  0001 C CNN
-	1    13600 4850
-	-1   0    0    1
-$EndComp
-$Comp
-L device:R R14
-U 1 1 5AE1E349
-P 13900 4350
-F 0 "R14" H 13970 4396 50  0000 L CNN
-F 1 "9.1k" V 13900 4250 50  0000 L CNN
-F 2 "Resistors_THT:R_Axial_DIN0207_L6.3mm_D2.5mm_P7.62mm_Horizontal" V 13830 4350 50  0001 C CNN
-F 3 "" H 13900 4350 50  0001 C CNN
-	1    13900 4350
-	-1   0    0    1
-$EndComp
-$Comp
-L device:R R12
-U 1 1 5AE1E41D
-P 13600 4350
-F 0 "R12" H 13670 4396 50  0000 L CNN
-F 1 "9.1k" V 13600 4250 50  0000 L CNN
-F 2 "Resistors_THT:R_Axial_DIN0207_L6.3mm_D2.5mm_P7.62mm_Horizontal" V 13530 4350 50  0001 C CNN
-F 3 "" H 13600 4350 50  0001 C CNN
-	1    13600 4350
-	-1   0    0    1
-$EndComp
-Wire Wire Line
-	13900 4700 13900 4550
-Wire Wire Line
-	13600 4700 13600 4650
-Wire Wire Line
-	13600 4200 13600 4150
-Wire Wire Line
-	13600 4150 14850 4150
-Wire Wire Line
-	13900 4200 14350 4200
-Wire Wire Line
-	14350 4200 14350 4350
-Wire Wire Line
-	14350 4350 14850 4350
-$Comp
-L power:GND #PWR013
-U 1 1 5AE5E820
-P 13900 5000
-F 0 "#PWR013" H 13900 4750 50  0001 C CNN
-F 1 "GND" H 13905 4827 50  0000 C CNN
-F 2 "" H 13900 5000 50  0001 C CNN
-F 3 "" H 13900 5000 50  0001 C CNN
-	1    13900 5000
-	1    0    0    -1
-$EndComp
-$Comp
-L power:GND #PWR012
-U 1 1 5AE5E8F4
-P 13600 5000
-F 0 "#PWR012" H 13600 4750 50  0001 C CNN
-F 1 "GND" H 13605 4827 50  0000 C CNN
-F 2 "" H 13600 5000 50  0001 C CNN
-F 3 "" H 13600 5000 50  0001 C CNN
-	1    13600 5000
-	1    0    0    -1
-$EndComp
-Text GLabel 13050 4550 0    50   Input ~ 0
-L_OUT
-Text GLabel 13050 4650 0    50   Input ~ 0
-R_OUT
-Wire Wire Line
-	13050 4550 13900 4550
-Connection ~ 13900 4550
-Wire Wire Line
-	13900 4550 13900 4500
-Wire Wire Line
-	13050 4650 13600 4650
-Connection ~ 13600 4650
-Wire Wire Line
-	13600 4650 13600 4500
+Wire Wire Line
+	14750 4750 14750 4650
+Wire Wire Line
+	14750 4650 14850 4650
 Text GLabel 950  3550 0    50   Input ~ 0
 SD_MOSI
@@
 	8700 10300 8700 7700
 Wire Notes Line
-	8700 7700 2350 7700
-Wire Notes Line
-	2350 7700 2350 10300
+	2250 7700 2250 10300
 Text Notes 4650 4650 0    50   ~ 0
 Main Soundchips, CPU, RAM & COM
@@
 Wire Wire Line
 	8050 2950 7800 2950
+$Comp
+L device:POT_Dual RV1
+U 1 1 5AE727F6
+P 14250 4400
+F 0 "RV1" V 14204 4212 50  0000 R CNN
+F 1 "POT_Dual" V 14295 4212 50  0000 R CNN
+F 2 "Potentiometers:Potentiometer_Alps_RK163_Double_Vertical" H 14500 4325 50  0001 C CNN
+F 3 "" H 14500 4325 50  0001 C CNN
+	1    14250 4400
+	0    1    1    0
+$EndComp
+Wire Wire Line
+	13550 4000 14150 4000
+Wire Wire Line
+	13550 4500 14150 4500
+$Comp
+L power:GND #PWR012
+U 1 1 5AE8AAD8
+P 14150 4300
+F 0 "#PWR012" H 14150 4050 50  0001 C CNN
+F 1 "GND" H 14155 4127 50  0000 C CNN
+F 2 "" H 14150 4300 50  0001 C CNN
+F 3 "" H 14150 4300 50  0001 C CNN
+	1    14150 4300
+	1    0    0    -1
+$EndComp
+$Comp
+L power:GND #PWR013
+U 1 1 5AE8ABA4
+P 14150 4800
+F 0 "#PWR013" H 14150 4550 50  0001 C CNN
+F 1 "GND" H 14155 4627 50  0000 C CNN
+F 2 "" H 14150 4800 50  0001 C CNN
+F 3 "" H 14150 4800 50  0001 C CNN
+	1    14150 4800
+	1    0    0    -1
+$EndComp
+Wire Wire Line
+	14350 4650 14450 4650
+Wire Wire Line
+	14450 4350 14850 4350
+Wire Wire Line
+	14450 4350 14450 4650
+Wire Wire Line
+	14350 4150 14850 4150
+$Comp
+L device:CP1_Small C37
+U 1 1 5AEBE891
+P 5700 2850
+F 0 "C37" V 5928 2850 50  0000 C CNN
+F 1 "1000uF" V 5837 2850 50  0000 C CNN
+F 2 "Capacitors_THT:CP_Radial_D8.0mm_P2.50mm" H 5700 2850 50  0001 C CNN
+F 3 "" H 5700 2850 50  0001 C CNN
+	1    5700 2850
+	0    -1   -1   0
+$EndComp
+Wire Wire Line
+	5600 2850 5550 2850
+Connection ~ 5550 2850
+Wire Wire Line
+	5550 2850 5550 3150
+$Comp
+L power:GND #PWR014
+U 1 1 5AECA9B3
+P 5800 2850
+F 0 "#PWR014" H 5800 2600 50  0001 C CNN
+F 1 "GND" V 5805 2722 50  0000 R CNN
+F 2 "" H 5800 2850 50  0001 C CNN
+F 3 "" H 5800 2850 50  0001 C CNN
+	1    5800 2850
+	0    -1   -1   0
+$EndComp
+Wire Wire Line
+	5550 2550 5550 2850
+$Comp
+L power:GND #PWR?
+U 1 1 5AEDE0C9
+P 10000 2250
+F 0 "#PWR?" H 10000 2000 50  0001 C CNN
+F 1 "GND" V 10005 2122 50  0000 R CNN
+F 2 "" H 10000 2250 50  0001 C CNN
+F 3 "" H 10000 2250 50  0001 C CNN
+	1    10000 2250
+	0    1    1    0
+$EndComp
+Wire Notes Line
+	2250 7700 8700 7700
 $EndSCHEMATC

Commit message: PCB Complete
Connections:
- wire segments 217 -> 216
Changed lines of the file:
@@
 Connection ~ 2900 3050
 Connection ~ 3100 2950
-Wire Wire Line
-	2700 2950 2900 2950
 $Comp
 L power:GND #PWR0129
@@
 Text Notes 12350 5250 0    50   ~ 0
 Pre-amp
-Connection ~ 2900 2950
-Wire Wire Line
-	2900 2950 3100 2950
 Wire Notes Line
 	2250 10300 8700 10300
@@
 	5550 2550 5550 2850
 $Comp
-L power:GND #PWR?
+L power:GND #PWR0156
 U 1 1 5AEDE0C9
 P 10000 2250
-F 0 "#PWR?" H 10000 2000 50  0001 C CNN
+F 0 "#PWR0156" H 10000 2000 50  0001 C CNN
 F 1 "GND" V 10005 2122 50  0000 R CNN
 F 2 "" H 10000 2250 50  0001 C CNN
@@
 Wire Notes Line
 	2250 7700 8700 7700
+Wire Wire Line
+	2700 2950 3100 2950
 $EndSCHEMATC
