File: Schematics/STM32_MegaBlaster/STM32_MegaBlaster.sch (KiCad schematic (older format))
At the start: 86 parts, among them J1 SD_Card, J2 USB_B, J3 Barrel_Jack, J4 AMP_OUT, SW1 PREV, SW2 RAND, SW3 NEXT, SW4 OPTION, SW5 POWER, SW6 MUTE PSG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

Commit message: Added interactive HTML BOM guide
Parts:
- C20, C21: symbol Device:C_Small -> STM32_MegaBlaster-rescue:C_Small-Device
Changed lines of the file:
@@
 Connection ~ 12600 7150
 $Comp
-L Device:C_Small C20
+L STM32_MegaBlaster-rescue:C_Small-Device C20
 U 1 1 5AEDFA79
 P 13000 6300
@@
 	12600 6300 12900 6300
 $Comp
-L Device:C_Small C21
+L STM32_MegaBlaster-rescue:C_Small-Device C21
 U 1 1 5AEE7909
 P 13000 7150

Commit message: Fixed SN76489 typo on schematic
Parts:
- RV1: symbol device:POT_Dual -> STM32_MegaBlaster-rescue:POT_Dual-device
- U2: value SN769486 -> SN76489
Changed lines of the file:
@@
 P 4600 2200
 F 0 "U2" H 4675 3087 60  0000 C CNN
-F 1 "SN769486" H 4675 2981 60  0000 C CNN
+F 1 "SN76489" H 4675 2981 60  0000 C CNN
 F 2 "Housings_DIP:DIP-16_W7.62mm" H 4550 1900 60  0001 C CNN
 F 3 "" H 4550 1900 60  0001 C CNN
@@
 	8050 2950 7800 2950
 $Comp
-L device:POT_Dual RV1
+L STM32_MegaBlaster-rescue:POT_Dual-device RV1
 U 1 1 5AE727F6
 P 14250 4400
