File: Schematics/STM32_MegaBlaster/STM32_MegaBlaster.sch (KiCad schematic (older format))
At the start: 86 parts, among them J1 SD_Card, J2 USB_B, J3 Barrel_Jack, J4 AMP_OUT, SW1 PREV, SW2 RAND, SW3 NEXT, SW4 OPTION, SW5 POWER, SW6 MUTE PSG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

Commit message: Schematic correction
Parts:
- C20, C21: symbol STM32_MegaBlaster-rescue:C_Small-Device -> STM32_MegaBlaster-rescue:C_Small-Device-STM32_MegaBlaster-rescue
- C33, C35: value 68nF -> 0.68uF
- L4, L5: value 2.2mH -> 22uH
- RV1: symbol STM32_MegaBlaster-rescue:POT_Dual-device -> STM32_MegaBlaster-rescue:POT_Dual-device-STM32_MegaBlaster-rescue
- U2: symbol sn76489:SN76489 -> STM32_MegaBlaster-rescue:SN76489-sn76489
Changed lines of the file:
@@
 $EndComp
 $Comp
-L sn76489:SN76489 U2
+L STM32_MegaBlaster-rescue:SN76489-sn76489 U2
 U 1 1 5ADCFD43
 P 4600 2200
@@
 Connection ~ 12600 7150
 $Comp
-L STM32_MegaBlaster-rescue:C_Small-Device C20
+L STM32_MegaBlaster-rescue:C_Small-Device-STM32_MegaBlaster-rescue C20
 U 1 1 5AEDFA79
 P 13000 6300
@@
 	12600 6300 12900 6300
 $Comp
-L STM32_MegaBlaster-rescue:C_Small-Device C21
+L STM32_MegaBlaster-rescue:C_Small-Device-STM32_MegaBlaster-rescue C21
 U 1 1 5AEE7909
 P 13000 7150
@@
 P 12550 2250
 F 0 "L4" V 12600 2250 50  0000 C CNN
-F 1 "2.2mH" V 12500 2200 50  0000 C CNN
+F 1 "22uH" V 12500 2200 50  0000 C CNN
 F 2 "Inductors_THT:L_Radial_D8.7mm_P5.00mm_Fastron_07HCP" H 12550 2250 50  0001 C CNN
 F 3 "" H 12550 2250 50  0001 C CNN
@@
 P 12800 2150
 F 0 "C33" H 12892 2196 50  0000 L CNN
-F 1 "68nF" H 12892 2105 50  0000 L CNN
+F 1 "0.68uF" H 12892 2105 50  0000 L CNN
 F 2 "Capacitors_THT:C_Disc_D3.0mm_W1.6mm_P2.50mm" H 12800 2150 50  0001 C CNN
 F 3 "" H 12800 2150 50  0001 C CNN
@@
 	8050 2950 7800 2950
 $Comp
-L STM32_MegaBlaster-rescue:POT_Dual-device RV1
+L STM32_MegaBlaster-rescue:POT_Dual-device-STM32_MegaBlaster-rescue RV1
 U 1 1 5AE727F6
 P 14250 4400
@@
 P 12600 2950
 F 0 "L5" V 12785 2950 50  0000 C CNN
-F 1 "2.2mH" V 12694 2950 50  0000 C CNN
+F 1 "22uH" V 12694 2950 50  0000 C CNN
 F 2 "Inductors_THT:L_Radial_D8.7mm_P5.00mm_Fastron_07HCP" H 12600 2950 50  0001 C CNN
 F 3 "" H 12600 2950 50  0001 C CNN
@@
 P 12800 3050
 F 0 "C35" H 12892 3096 50  0000 L CNN
-F 1 "68nF" H 12892 3005 50  0000 L CNN
+F 1 "0.68uF" H 12892 3005 50  0000 L CNN
 F 2 "Capacitors_THT:CP_Radial_D6.3mm_P2.50mm" H 12800 3050 50  0001 C CNN
 F 3 "" H 12800 3050 50  0001 C CNN

Commit message: New VGM Engine, yay!
Parts:
- C1, C10, C11, C12, C15, C16, C19, C2, C22, C23, C24, C25, C26, C3, C31, C32, C33, C35, C38, C4, C5, C6, C7, C9: symbol device:C_Small -> STM32_MegaBlaster-rescue:C_Small-device
- C13, C14, C17, C18, C27, C28, C29, C30, C34, C36, C37, C8: symbol device:CP1_Small -> STM32_MegaBlaster-rescue:CP1_Small-device
- D1: symbol device:D_Schottky_Small_ALT -> STM32_MegaBlaster-rescue:D_Schottky_Small_ALT-device
- J1: symbol conn:SD_Card -> STM32_MegaBlaster-rescue:SD_Card-conn
- J2: symbol conn:USB_B -> STM32_MegaBlaster-rescue:USB_B-conn
- J3: symbol conn:Barrel_Jack -> STM32_MegaBlaster-rescue:Barrel_Jack-conn
- L1, L2, L3, L4, L5: symbol device:L_Small -> STM32_MegaBlaster-rescue:L_Small-device
- R1, R10, R11, R2, R24, R25, R26, R27, R28, R29, R3, R30, R4, R5, R6, R7, R8, R9: symbol device:R -> STM32_MegaBlaster-rescue:R-device
- SW1, SW2, SW3, SW4: symbol switches:SW_Push_Dual -> STM32_MegaBlaster-rescue:SW_Push_Dual-switches
- SW5: symbol switches:SW_SPST -> STM32_MegaBlaster-rescue:SW_SPST-switches
- SW6: symbol switches:SW_Push_SPDT -> STM32_MegaBlaster-rescue:SW_Push_SPDT-switches
- U10: symbol regul:LD1117S33TR_SOT223 -> STM32_MegaBlaster-rescue:LD1117S33TR_SOT223-regul
- U11: symbol dc-dc:LM2596T-5 -> STM32_MegaBlaster-rescue:LM2596T-5-dc-dc
- U8: symbol linear:TL062 -> STM32_MegaBlaster-rescue:TL062-linear
- Y1: symbol device:Crystal_Small -> STM32_MegaBlaster-rescue:Crystal_Small-device
