File: Schematics/STM32_MegaBlaster/STM32_MegaBlaster.kicad_pcb (KiCad board)
At the start: 2 copper layers, 138.4 x 91.4 mm, 91 parts, among them J1 SD_Card, J2 USB_B, J3 Barrel_Jack, J4 AMP_OUT, SW5 POWER, SW6 MUTE PSG, U1 BluePill_STM32F103C, U10 LD1117S33, U11 LM2596T-5, U12 I2C_OLED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

Commit message: Fixed SN76489 typo on schematic
Parts:
- U2: value SN769486 -> SN76489
Changed lines of the file:
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@@
-(kicad_pcb (version 20171130) (host pcbnew "(5.0.0-rc2-dev-493-gd776eaca8)")
+(kicad_pcb (version 20171130) (host pcbnew "(5.0.2)-1")
   (general
     (thickness 1.6)
@@
     (pad_drill 1.2)
     (pad_to_mask_clearance 0.2)
+    (solder_mask_min_width 0.25)
     (aux_axis_origin 0 0)
     (visible_elements 7FFFFFFF)
@@
       (hpglpennumber 1)
       (hpglpenspeed 20)
-      (hpglpendiameter 15)
+      (hpglpendiameter 15.000000)
       (psnegative false)
       (psa4output false)
@@
       (drillshape 0)
       (scaleselection 1)
-      (outputdirectory Megablaster_Gerber/))
+      (outputdirectory "Megablaster_Gerber/"))
   )
   (net 0 "")
@@
       (effects (font (size 1 1) (thickness 0.15)))
     )
-    (fp_text value SN769486 (at 3.81 20.11 90) (layer F.Fab)
+    (fp_text value SN76489 (at 3.81 20.11 90) (layer F.Fab)
       (effects (font (size 1 1) (thickness 0.15)))
     )

Commit message: New meta file remover function to prevent crashs from system files.
Parts:
- added H1: MountingHole_3.2mm_M3, Mounting_Holes:MountingHole_3.2mm_M3, F.Cu at (100.3, 38.1)
- added H1: MountingHole_3.2mm_M3, Mounting_Holes:MountingHole_3.2mm_M3, F.Cu at (132.7, 83.8)
- added H1: MountingHole_3.2mm_M3, Mounting_Holes:MountingHole_3.2mm_M3, F.Cu at (183.5, 33.7)
- added H1: MountingHole_3.2mm_M3, Mounting_Holes:MountingHole_3.2mm_M3, F.Cu at (172.7, 117.5)
- added H1: MountingHole_3.2mm_M3, Mounting_Holes:MountingHole_3.2mm_M3, F.Cu at (62.9, 117.5)
- moved J3 1.91 mm to (192.4, 44.5)
Routing:
- net Net-(J1-Pad12): track 94.3 -> 0.00 mm
- net GND: track 73.6 -> 77.2 mm, vias 11 -> 31
- net I2C_SDA: track 239.6 -> 242.5 mm
- net I2C_SCL: track 197.6 -> 199.5 mm
- net Net-(J3-Pad1): track 8.28 -> 9.07 mm
Other:
- board text added: "Revision 2b"
- board text removed: "Revision 2"
